File: _autosave-bkm-129x-simple.kicad_pcb (KiCad board)
At the start: 2 copper layers, 105 x 160 mm, 65 parts, among them J1 YG_IN, J11 YG_OUT, J2 PBB_IN, J21 PBB_OUT, J3 PRR_IN, J31 PRR_OUT, J4 SYNC_IN, J41 SYNC_OUT, J5 Conn_02x32_Row_Letter_Last, J6 ICSP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

Commit message: redrawn, thanks skum
Other:
- board text added: "BKM 129X clone 2021-08-18 rev 1.0 jam@wakabavideo.com code and original design by Martin Hejnfelt www.immerhax.com"
- board text removed: "(2020-2021) Martin Hejnfelt (martin@hejnfelt.com) www.immerhax.com"
- board text removed: "Rev. C"
Changed lines of the file:
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@@
   (general
     (thickness 1.6)
-    (drawings 24)
+    (drawings 23)
     (tracks 613)
     (zones 0)
@@
     (effects (font (size 1.5 1.5) (thickness 0.3)))
   )
-  (gr_text "Rev. C" (at 194.564 201.676) (layer F.SilkS)
-    (effects (font (size 1.5 1.5) (thickness 0.3)))
-  )
   (gr_text "SYNC IN" (at 110.6 168.4 90) (layer F.SilkS)
     (effects (font (size 1.5 1.5) (thickness 0.3)))
@@
     (effects (font (size 1.5 1.5) (thickness 0.3)))
   )
-  (gr_text "(2020-2021) Martin Hejnfelt (martin@hejnfelt.com)\nwww.immerhax.com" (at 152.4 199.644) (layer F.SilkS)
-    (effects (font (size 1.5 1.5) (thickness 0.3)))
+  (gr_text "BKM 129X clone\n2021-08-18 rev 1.0\njam@wakabavideo.com\ncode and original design by Martin Hejnfelt www.immerhax.com" (at 198.15 197.3) (layer F.SilkS)
+    (effects (font (size 1.5 1.5) (thickness 0.3)) (justify right))
   )
-  (gr_text "BKM-129X Compatible" (at 152.4 45.212) (layer F.SilkS)
-    (effects (font (size 1.5 1.5) (thickness 0.3)))
+  (gr_text "BKM-129X Compatible" (at 152.25 55.15) (layer F.SilkS)
+    (effects (font (size 3 3) (thickness 0.5)))
   )
   (gr_line (start 103.579 123.4015) (end 107.643 123.4015) (angle 90) (layer F.SilkS) (width 0.2))
