File: _autosave-bkm-129x-simple.sch (KiCad schematic (older format))
At the start: 58 parts, among them J1 YG_IN, J11 YG_OUT, J2 PBB_IN, J21 PBB_OUT, J3 PRR_IN, J31 PRR_OUT, J4 SYNC_IN, J41 SYNC_OUT, J5 Conn_02x32_Row_Letter_Last, Q1 DTC144EKAT146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

Commit message: redrawn, thanks skum
Parts:
- added FID1: Fiducial, videobits:borgar, symbol Mechanical:Fiducial
- gave numbers to parts that had none: 2
Changed lines of the file:
@@
 $EndComp
 $Comp
-L bkm-129x-simple-rescue:C-bkm-129x-simple-rescue C?
+L bkm-129x-simple-rescue:C-bkm-129x-simple-rescue C9
 U 1 1 612C1DDF
 P 8350 4250
-F 0 "C?" H 8375 4350 50  0000 L CNN
+F 0 "C9" H 8375 4350 50  0000 L CNN
 F 1 "0.1uF" H 8375 4150 50  0000 L CNN
 F 2 "Capacitor_SMD:C_0805_2012Metric_Pad1.18x1.45mm_HandSolder" H 8388 4100 50  0001 C CNN
@@
 $EndComp
 $Comp
-L power:GNDA #PWR?
+L power:GNDA #PWR0118
 U 1 1 612C1DE5
 P 8200 4250
-F 0 "#PWR?" H 8200 4000 50  0001 C CNN
+F 0 "#PWR0118" H 8200 4000 50  0001 C CNN
 F 1 "GNDA" V 8200 4050 50  0000 C CNN
 F 2 "" H 8200 4250 50  0001 C CNN
@@
 $EndComp
 $Comp
-L power:+3.3V #PWR?
+L power:+3.3V #PWR0119
 U 1 1 612C1DEB
 P 8500 4250
-F 0 "#PWR?" H 8500 4100 50  0001 C CNN
+F 0 "#PWR0119" H 8500 4100 50  0001 C CNN
 F 1 "+3.3V" V 8500 4500 50  0000 C CNN
 F 2 "" H 8500 4250 50  0001 C CNN
@@
 $EndComp
 $Comp
-L bkm-129x-simple-rescue:C-bkm-129x-simple-rescue C?
+L bkm-129x-simple-rescue:C-bkm-129x-simple-rescue C8
 U 1 1 612CE495
 P 7800 4600
-F 0 "C?" H 7825 4700 50  0000 L CNN
+F 0 "C8" H 7825 4700 50  0000 L CNN
 F 1 "0.1uF" H 7825 4500 50  0000 L CNN
 F 2 "Capacitor_SMD:C_0805_2012Metric_Pad1.18x1.45mm_HandSolder" H 7838 4450 50  0001 C CNN
@@
 $EndComp
 $Comp
-L power:GNDA #PWR?
+L power:GNDA #PWR0120
 U 1 1 612CE49B
 P 7650 4600
-F 0 "#PWR?" H 7650 4350 50  0001 C CNN
+F 0 "#PWR0120" H 7650 4350 50  0001 C CNN
 F 1 "GNDA" V 7650 4400 50  0000 C CNN
 F 2 "" H 7650 4600 50  0001 C CNN
@@
 $EndComp
 $Comp
-L power:+3.3V #PWR?
+L power:+3.3V #PWR0121
 U 1 1 612CE4A1
 P 7950 4600
-F 0 "#PWR?" H 7950 4450 50  0001 C CNN
+F 0 "#PWR0121" H 7950 4450 50  0001 C CNN
 F 1 "+3.3V" V 7950 4850 50  0000 C CNN
 F 2 "" H 7950 4600 50  0001 C CNN
@@
 	0    1    1    0
 $EndComp
+$Comp
+L Mechanical:Fiducial FID1
+U 1 1 6135E536
+P 9350 6250
+F 0 "FID1" H 9435 6296 50  0000 L CNN
+F 1 "Fiducial" H 9435 6205 50  0000 L CNN
+F 2 "videobits:borgar" H 9350 6250 50  0001 C CNN
+F 3 "~" H 9350 6250 50  0001 C CNN
+	1    9350 6250
+	1    0    0    -1
+$EndComp
 $EndSCHEMATC
